File: Kicad/PMA5-123-3W_DConly/PMA5-123-3W_DConly_v1.kicad_pcb (KiCad board)
At the start: 2 copper layers, 40 x 43 mm, 42 parts, among them J1 8V-DC, J2 UPDI, J3 RF_unit, Q1 FMG1, Q2 BC850, SW1 SW_Push, U1 L78L05_SOT89, U2 R05C1TF05S-R, U3 MIC29302, U5 INA168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

Commit message: Update Kicad and SW
Parts:
- removed R14: 10K, Resistor_SMD:R_0603_1608Metric
- added R8: 10K, Resistor_SMD:R_0603_1608Metric, F.Cu at (179.3, 91.0)
- C1: value 100n -> 10u; footprint Capacitor_SMD:C_0603_1608Metric -> Capacitor_SMD:C_0805_2012Metric
- C12, C2, C5: footprint Capacitor_SMD:C_0805_2012Metric -> Capacitor_SMD:C_0603_1608Metric
- C23: value 100n -> 1n
- Q2: value BC850 -> BC859C
- R1: value 0.05R -> 0.1R
- R3: value 22K -> 2K2
- R4: value 4K7 -> 470R
- R6: value 27K -> 5K1
- R7: value 10K -> 2K
- R9: value 10K -> 100K
- moved C23 7.80 mm to (161.5, 74.1)
- moved R2 0.86 mm to (170.7, 86.1), turned to 0 degrees
- moved D4 0.20 mm to (183.5, 93.1)
- moved R12 0.20 mm to (183.5, 89.8)
- turned C5 to -90 degrees
Connections:
- C1 pad 1: Net-(C3-Pad1) -> Net-(C1-Pad1)
- C3 pad 1: Net-(C3-Pad1) -> Net-(C1-Pad1)
- C5 pad 1: GNDREF -> Net-(C5-Pad1)
- C5 pad 2: Net-(C5-Pad2) -> GNDREF
- D1 pad 1: Net-(C3-Pad1) -> Net-(C1-Pad1)
- F1 pad 2: Net-(C3-Pad1) -> Net-(C1-Pad1)
- Q1 pad 2: Net-(Q1-Pad2) -> unconnected-(Q1-Pad2)
- Q1 pad 3: Net-(Q1-Pad3) -> unconnected-(Q1-Pad3)
- Q2 pad 3: Net-(C5-Pad2) -> Net-(C5-Pad1)
- R10 pad 2: Net-(C23-Pad1) -> Net-(R10-Pad2)
- R12 pad 1: Net-(C5-Pad2) -> Net-(C5-Pad1)
- R2 pad 1: Net-(C3-Pad1) -> Net-(R2-Pad1)
- R2 pad 2: Net-(Q1-Pad2) -> GNDREF
- R7 pad 2: Net-(C5-Pad2) -> Net-(C5-Pad1)
- R9 pad 1: Net-(R9-Pad1) -> Net-(C23-Pad1)
- U1 pad 3: Net-(C3-Pad1) -> Net-(C1-Pad1)
- U2 pad 10: Net-(C5-Pad2) -> Net-(C5-Pad1)
- U2 pad 11: Net-(C5-Pad2) -> Net-(C5-Pad1)
- U2 pad 12: Net-(C5-Pad2) -> Net-(C5-Pad1)
- U2 pad 7: GNDREF -> Net-(C5-Pad1)
- U3 pad 1: Net-(Q1-Pad2) -> Net-(R2-Pad1)
- U3 pad 2: Net-(C3-Pad1) -> Net-(C1-Pad1)
- U5 pad 1: Net-(R9-Pad1) -> Net-(C23-Pad1)
- U6 pad 3: Net-(R9-Pad1) -> Net-(C23-Pad1)
- U6 pad 5: Net-(Q1-Pad3) -> Net-(R2-Pad1)
- U6 pad 6: Net-(C23-Pad1) -> Net-(R10-Pad2)
Routing:
- net Net-(C1-Pad1): track 0.00 -> 44.5 mm, vias 0 -> 2
- net Net-(C3-Pad1): track 42.9 -> 0.00 mm, vias 2 -> 0
- net Net-(C5-Pad2): track 39.9 -> 0.00 mm, vias 4 -> 0
- net Net-(C5-Pad1): track 0.00 -> 37.7 mm, vias 0 -> 4
- net Net-(R2-Pad1): track 0.00 -> 26.7 mm, vias 0 -> 2
- net Net-(Q1-Pad3): track 22.1 -> 0.00 mm
- net Net-(R9-Pad1): track 19.7 -> 0.00 mm, vias 2 -> 0
- net Net-(C23-Pad1): track 4.70 -> 20.9 mm, vias 0 -> 2
- net Net-(Q1-Pad2): track 14.7 -> 0.00 mm, vias 2 -> 0
- net Net-(C22-Pad1): track 7.07 -> 10.5 mm
- net Net-(R10-Pad2): track 0.00 -> 2.25 mm
- net +5V: track 42.6 -> 41.1 mm
- net GNDREF: track 42.0 -> 42.1 mm, vias 80 -> 82

Commit message: Added R13 and JP1
Parts:
- added JP1: ', Jumper:SolderJumper-2_P1.3mm_Open_RoundedPad1.0x1.5mm, F.Cu at (158.8, 60.8)
- added R13: 100R, Resistor_SMD:R_0603_1608Metric, F.Cu at (180.2, 59.6)
- C23: value 1n -> Opt
- D2: value LED -> Blue LED opt
- D3: value LED -> Red LED
- D4: value LED -> Green LED
- R12: value 180R -> 330R
- R5: value 330R -> 10K opt
- R9: value 100K -> 51K
Routing:
- net Net-(R5-Pad1): track 19.4 -> 22.9 mm
- net Net-(J3-Pad3): track 10.6 -> 14.1 mm
- net GNDREF: vias 82 -> 83
Changed lines of the file:
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@@
       (effects (font (size 1 1) (thickness 0.15)))
     )
-    (fp_text value "180R" (at 0 1.43 90) (layer "F.Fab")
+    (fp_text value "330R" (at 0 1.43 90) (layer "F.Fab")
       (effects (font (size 1 1) (thickness 0.15)))
     )
@@
     (property "Sheetname" "")
     (attr smd)
-    (fp_text reference "U5" (at 3.55 0 180) (layer "F.SilkS")
+    (fp_text reference "U5" (at 3.95 2.1 180) (layer "F.SilkS")
       (effects (font (size 1 1) (thickness 0.15)))
     )
@@
       (effects (font (size 1 1) (thickness 0.15)))
     )
-    (fp_text value "LED" (at 0 1.65 90) (layer "F.Fab")
+    (fp_text value "Red LED" (at 0 1.65 90) (layer "F.Fab")
       (effects (font (size 1 1) (thickness 0.15)))
     )
@@
     )
   )
+  (footprint "Jumper:SolderJumper-2_P1.3mm_Open_RoundedPad1.0x1.5mm" (layer "F.Cu")
+    (at 158.8 60.75 -90)
+    (descr "SMD Solder Jumper, 1x1.5mm, rounded Pads, 0.3mm gap, open")
+    (tags "solder jumper open")
+    (property "Sheetfile" "PMA5-123-3W_DConly_v1.kicad_sch")
+    (property "Sheetname" "")
+    (attr exclude_from_pos_files)
+    (fp_text reference "JP1" (at 0 -1.8 90) (layer "F.SilkS")
+      (effects (font (size 1 1) (thickness 0.15)))
+    )
+    (fp_text value "'" (at 0 1.9 90) (layer "F.Fab")
+      (effects (font (size 1 1) (thickness 0.15)))
+    )
+    (fp_line (start -0.7 -1) (end 0.7 -1) (layer "F.SilkS") (width 0.12))
+    (fp_line (start 0.7 1) (end -0.7 1) (layer "F.SilkS") (width 0.12))
+    (fp_line (start 1.4 -0.3) (end 1.4 0.3) (layer "F.SilkS") (width 0.12))
+    (fp_line (start -1.4 0.3) (end -1.4 -0.3) (layer "F.SilkS") (width 0.12))
+    (fp_arc (start -1.4 -0.3) (mid -1.194975 -0.794975) (end -0.7 -1) (layer "F.SilkS") (width 0.12))
+    (fp_arc (start -0.7 1) (mid -1.194975 0.794975) (end -1.4 0.3) (layer "F.SilkS") (width 0.12))
+    (fp_arc (start 0.7 -1) (mid 1.194975 -0.794975) (end 1.4 -0.3) (layer "F.SilkS") (width 0.12))
+    (fp_arc (start 1.4 0.3) (mid 1.194975 0.794975) (end 0.7 1) (layer "F.SilkS") (width 0.12))
+    (fp_line (start -1.65 -1.25) (end 1.65 -1.25) (layer "F.CrtYd") (width 0.05))
+    (fp_line (start 1.65 1.25) (end 1.65 -1.25) (layer "F.CrtYd") (width 0.05))
+    (fp_line (start -1.65 -1.25) (end -1.65 1.25) (layer "F.CrtYd") (width 0.05))
+    (fp_line (start 1.65 1.25) (end -1.65 1.25) (layer "F.CrtYd") (width 0.05))
+    (pad "1" smd custom (at -0.65 0 270) (size 1 0.5) (layers "F.Cu" "F.Mask")
+      (net 1 "GNDREF") (pinfunction "A") (pintype "passive") (zone_connect 2)
+      (options (clearance outline) (anchor rect))
+      (primitives
+        (gr_circle (center 0 0.25) (end 0.5 0.25) (width 0) (fill yes))
+        (gr_circle (center 0 -0.25) (end 0.5 -0.25) (width 0) (fill yes))
+        (gr_poly (pts
+            (xy 0.5 0.75)
+            (xy 0 0.75)
+            (xy 0 -0.75)
+            (xy 0.5 -0.75)
+          ) (width 0) (fill yes))
+      ))
+    (pad "2" smd custom (at 0.65 0 270) (size 1 0.5) (layers "F.Cu" "F.Mask")
+      (net 16 "Net-(R5-Pad1)") (pinfunction "B") (pintype "passive") (zone_connect 2)
+      (options (clearance outline) (anchor rect))
+      (primitives
+        (gr_circle (center 0 0.25) (end 0.5 0.25) (width 0) (fill yes))
+        (gr_circle (center 0 -0.25) (end 0.5 -0.25) (width 0) (fill yes))
+        (gr_poly (pts
+            (xy 0 0.75)
+            (xy -0.5 0.75)
+            (xy -0.5 -0.75)
+            (xy 0 -0.75)
+          ) (width 0) (fill yes))
+      ))
+  )
   (footprint "Resistor_SMD:R_0603_1608Metric" (layer "F.Cu")
     (at 156.8 65.7 -90)
@@
       (effects (font (size 1 1) (thickness 0.15)))
     )
-    (fp_text value "330R" (at 0 1.43 90) (layer "F.Fab")
+    (fp_text value "10K opt" (at 0 1.43 90) (layer "F.Fab")
       (effects (font (size 1 1) (thickness 0.15)))
     )
@@
     )
   )
+  (footprint "Resistor_SMD:R_0603_1608Metric" (layer "F.Cu")
+    (at 180.2 59.6)
+    (descr "Resistor SMD 0603 (1608 Metric), square (rectangular) end terminal, IPC_7351 nominal, (Body size source: IPC-SM-782 page 72, https://www.pcb-3d.com/wordpress/wp-content/uploads/ipc-sm-782a_amendment_1_and_2.pdf), generated with kicad-footprint-generator")
+    (tags "resistor")
+    (property "Sheetfile" "PMA5-123-3W_DConly_v1.kicad_sch")
+    (property "Sheetname" "")
+    (attr smd)
+    (fp_text reference "R13" (at 0 -1.43) (layer "F.SilkS")
+      (effects (font (size 1 1) (thickness 0.15)))
+    )
+    (fp_text value "100R" (at 0 1.43) (layer "F.Fab")
+      (effects (font (size 1 1) (thickness 0.15)))
+    )
+    (fp_text user "${REFERENCE}" (at 0 0) (layer "F.Fab")
+      (effects (font (size 0.4 0.4) (thickness 0.06)))
+    )
+    (fp_line (start -0.237258 -0.5225) (end 0.237258 -0.5225) (layer "F.SilkS") (width 0.12))
+    (fp_line (start -0.237258 0.5225) (end 0.237258 0.5225) (layer "F.SilkS") (width 0.12))
+    (fp_line (start -1.48 -0.73) (end 1.48 -0.73) (layer "F.CrtYd") (width 0.05))
+    (fp_line (start 1.48 0.73) (end -1.48 0.73) (layer "F.CrtYd") (width 0.05))
+    (fp_line (start -1.48 0.73) (end -1.48 -0.73) (layer "F.CrtYd") (width 0.05))
+    (fp_line (start 1.48 -0.73) (end 1.48 0.73) (layer "F.CrtYd") (width 0.05))
+    (fp_line (start -0.8 0.4125) (end -0.8 -0.4125) (layer "F.Fab") (width 0.1))
+    (fp_line (start 0.8 0.4125) (end -0.8 0.4125) (layer "F.Fab") (width 0.1))
+    (fp_line (start -0.8 -0.4125) (end 0.8 -0.4125) (layer "F.Fab") (width 0.1))
+    (fp_line (start 0.8 -0.4125) (end 0.8 0.4125) (layer "F.Fab") (width 0.1))
+    (pad "1" smd roundrect (at -0.825 0) (size 0.8 0.95) (layers "F.Cu" "F.Paste" "F.Mask") (roundrect_rratio 0.25)
+      (net 13 "Net-(J3-Pad3)") (pintype "passive"))
+    (pad "2" smd roundrect (at 0.825 0) (size 0.8 0.95) (layers "F.Cu" "F.Paste" "F.Mask") (roundrect_rratio 0.25)
+      (net 1 "GNDREF") (pintype "passive"))
+    (model "${KICAD6_3DMODEL_DIR}/Resistor_SMD.3dshapes/R_0603_1608Metric.wrl"
+      (offset (xyz 0 0 0))
+      (scale (xyz 1 1 1))
+      (rotate (xyz 0 0 0))
+    )
+  )
   (footprint "Capacitor_SMD:C_0603_1608Metric" (layer "F.Cu")
     (at 161.5 74.1 180)
@@
       (effects (font (size 1 1) (thickness 0.15)))
     )
-    (fp_text value "1n" (at 0 1.43) (layer "F.Fab")
+    (fp_text value "Opt" (at 0 1.43) (layer "F.Fab")
       (effects (font (size 1 1) (thickness 0.15)))
     )
@@
       (effects (font (size 1 1) (thickness 0.15)))
     )
-    (fp_text value "LED" (at 0 1.65 90) (layer "F.Fab")
+    (fp_text value "Blue LED opt" (at 0 1.65 90) (layer "F.Fab")
       (effects (font (size 1 1) (thickness 0.15)))
     )
@@
       (effects (font (size 1 1) (thickness 0.15)))
     )
-    (fp_text value "100K" (at 0 1.43) (layer "F.Fab")
+    (fp_text value "51K" (at 0 1.43) (layer "F.Fab")
       (effects (font (size 1 1) (thickness 0.15)))
     )
@@
       (effects (font (size 1 1) (thickness 0.15)))
     )
-    (fp_text value "LED" (at 0 1.65 90) (layer "F.Fab")
+    (fp_text value "Green LED" (at 0 1.65 90) (layer "F.Fab")
       (effects (font (size 1 1) (thickness 0.15)))
     )
@@
   (via (at 153.425 79.175) (size 0.8) (drill 0.4) (layers "F.Cu" "B.Cu") (net 1))
   (via (at 153.425 81.175) (size 0.8) (drill 0.4) (layers "F.Cu" "B.Cu") (net 1))
+  (via (at 181.9 59.6) (size 0.8) (drill 0.4) (layers "F.Cu" "B.Cu") (free) (net 1))
   (via (at 159.425 85.175) (size 0.8) (drill 0.4) (layers "F.Cu" "B.Cu") (net 1))
   (via (at 188 82.5) (size 0.8) (drill 0.4) (layers "F.Cu" "B.Cu") (free) (net 1))
@@
   (segment (start 163.5 73) (end 166 73) (width 0.5) (layer "B.Cu") (net 12))
   (segment (start 181.45 66.45) (end 184.7 66.45) (width 0.8) (layer "F.Cu") (net 13))
+  (segment (start 179.375 59.6) (end 179.275 59.5) (width 0.25) (layer "F.Cu") (net 13))
   (segment (start 176.75 61) (end 176.75 61.75) (width 0.8) (layer "F.Cu") (net 13))
   (segment (start 176.75 61.75) (end 181.45 66.45) (width 0.8) (layer "F.Cu") (net 13))
+  (segment (start 179.275 59.5) (end 176 59.5) (width 0.25) (layer "F.Cu") (net 13))
   (segment (start 175.265 74.33) (end 173.195 74.33) (width 0.5) (layer "F.Cu") (net 14))
   (segment (start 176.715 72.88) (end 175.265 74.33) (width 0.5) (layer "F.Cu") (net 14))
@@
   (segment (start 182.4 75.1) (end 181.188062 76.311938) (width 0.5) (layer "B.Cu") (net 15))
   (segment (start 169.01 68.1) (end 162.6 68.1) (width 0.5) (layer "F.Cu") (net 16))
+  (segment (start 161.7 64.9) (end 158.8 64.9) (width 0.5) (layer "F.Cu") (net 16))
   (segment (start 154.2 64.9) (end 153.6 65.5) (width 0.5) (layer "F.Cu") (net 16))
   (segment (start 169.79 67.32) (end 169.01 68.1) (width 0.5) (layer "F.Cu") (net 16))
-  (segment (start 161.7 64.9) (end 154.2 64.9) (width 0.5) (layer "F.Cu") (net 16))
+  (segment (start 158.8 61.4) (end 158.8 64.9) (width 0.25) (layer "F.Cu") (net 16))
+  (segment (start 158.8 64.9) (end 154.2 64.9) (width 0.5) (layer "F.Cu") (net 16))
   (via (at 162.6 68.1) (size 0.8) (drill 0.4) (layers "F.Cu" "B.Cu") (net 16))
   (via (at 161.7 64.9) (size 0.8) (drill 0.4) (layers "F.Cu" "B.Cu") (net 16))
