File: Kicad/PMA5-123-3W_DC_V1.0/PMA5-123-3W_DC_V1.0.kicad_sch (KiCad schematic)
At the start: 44 parts, among them J1 8V-DC, J2 UPDI, J3 RF_unit, Q1 FMG1, Q2 BC859C, SW1 SW_Push, U1 L78L05_SOT89, U2 R05C1TF05S-R, U3 MIC29302, U5 INA168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

Commit message: Update to version V1.0
Parts:
- D2: value Blue LED opt -> Blue LED
- R13: footprint Resistor_SMD:R_0603_1608Metric -> Resistor_SMD:R_0805_2012Metric
- R5: value 10K opt -> 10K
Other:
- note added: "1A => 1V"
- note removed: "1A => 2V"
- title: (none) -> PMA5-123-3W DC Controller
- moved on the sheet: C1, C12, C2, C21, C22, C23, C24, C3, C5, C9, D1, D2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
