File: Kicad/PMA5-123-3W_DC_V1.0/_autosave-PMA5-123-3W_DC_V1.0.kicad_pcb (KiCad board)
At the start: 2 copper layers, 40 x 43 mm, 44 parts, among them J1 8V-DC, J2 UPDI, J3 RF_unit, Q1 FMG1, Q2 BC859C, SW1 SW_Push, U1 L78L05_SOT89, U2 R05C1TF05S-R, U3 MIC29302, U5 INA168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

Commit message: Update to version V1.0
Parts:
- D2: value Blue LED opt -> Blue LED
- R13: footprint Resistor_SMD:R_0603_1608Metric -> Resistor_SMD:R_0805_2012Metric
- R5: value 10K opt -> 10K
- moved R8 7.63 mm to (176.1, 84.1), turned to -90 degrees
- moved C24 6.18 mm to (175.6, 66.6)
- moved R10 4.46 mm to (175.6, 71.3), turned to 90 degrees
- moved J2 1.63 mm to (178.7, 69.2)
- moved C22 1.41 mm to (178.6, 86.6)
- moved Q1 1.33 mm to (178.8, 83.2)
- moved R13 0.32 mm to (180.5, 59.5)
- moved C12 0.20 mm to (171.9, 81.3)
- moved C2 0.16 mm to (184.4, 79.0)
- moved C5 0.15 mm to (188.5, 73.5)
Routing:
- net GNDREF: track 42.1 -> 2.82 mm, vias 83 -> 81
- net Net-(R2-Pad1): track 26.7 -> 22.8 mm
- net Net-(C21-Pad2): track 19.1 -> 22.8 mm
- net Net-(R10-Pad2): track 2.25 -> 5.93 mm
- net Net-(C5-Pad1): track 37.7 -> 39.5 mm
- net Net-(J3-Pad3): track 14.1 -> 15.9 mm
- net Net-(C22-Pad1): track 10.5 -> 12.1 mm
- net Net-(JP1-Pad2): track 22.9 -> 24.1 mm
- net Net-(F1-Pad1): track 3.98 -> 3.15 mm
- net Net-(J2-Pad3): track 5.38 -> 4.65 mm
- net +5V: track 41.1 -> 41.6 mm
- net Net-(Q1-Pad1): track 11.5 -> 12.1 mm
- net Net-(C1-Pad1): track 44.5 -> 43.9 mm
- added copper zone on F.Cu, net +5V
- added copper zone on F.Cu, net Net-(C5-Pad1)
Other:
- board text added: "PCB V1.0"
